File: relays-hw/blinds.kicad_pcb (KiCad board)
At the start: 2 copper layers, 95.6 x 64.8 mm, 29 parts, among them J1 AC, J10 DC, J11 DTR, J12 DC, J2 DC, J4 SWITCH, J7 DRIVE, J8 CTS, J9 SERIAL, U1 ESP-12E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

Commit message: Revision 3
Parts:
- removed J4: SWITCH, Pin_Headers:Pin_Header_Straight_1x03_Pitch2.54mm
- removed R2: 1k, Resistors_SMD:R_0805_HandSoldering
- added J3: CH_PD, Pin_Headers:Pin_Header_Straight_1x01_Pitch2.54mm, F.Cu at (136.7, 126.7)
- C2: value 100nF -> 100uF; footprint Capacitors_SMD:C_0805_HandSoldering -> Capacitors_THT:CP_Radial_D6.3mm_P2.50mm
- J11: value DTR -> CH_PD
- J8: value CTS -> GPIO0
- PS1: footprint footprints:VTX-214-006 -> VTX-214-006
- R1: value 1k -> 10k
- RLY1: footprint footprint:relay_PE -> footprints:relay_PE
- U2: footprint footprints:LB1909MC_W -> footprints:LB1909MC
- moved REF** 113.3 mm to (179.3, 60.8), turned to 90 degrees
- moved REF** 113.3 mm to (179.3, 39.2), turned to 90 degrees
- moved J1 109.4 mm to (177.3, 51.5), turned to 90 degrees
- moved PS1 72.1 mm to (150.7, 44.5), turned to 180 degrees
- moved J12 39.9 mm to (132.6, 79.2), turned to 90 degrees
- moved J11 35.8 mm to (136.7, 121.0)
- moved REF** 33.4 mm to (120.9, 60.8), turned to 90 degrees
- moved REF** 33.3 mm to (120.9, 39.2), turned to 90 degrees
- moved J2 29.6 mm to (120.5, 49.2), turned to 0 degrees
- moved R1 3.30 mm to (135.1, 124.1), turned to 0 degrees
- moved C2 3.29 mm to (130.2, 91.1)
- moved J8 1.27 mm to (167.8, 110.2)
Connections:
- net /CTS renamed /GPIO0
- net /LED renamed /INT_LED
- net Net-(R5-Pad2) renamed /GPIO15
- J11 pad 1: /DTR -> /CH_PD
- R1 pad 1: /DTR -> VCC
- R1 pad 2: /WOES -> /RESET
- R3 pad 2: Net-(R3-Pad2) -> /CH_PD
- U1 pad 1: /DTR -> /RESET
- U1 pad 19: /GPIO9 -> Net-(U1-Pad19)
- U1 pad 20: /GPIO10 -> Net-(U1-Pad20)
- U1 pad 3: Net-(R3-Pad2) -> /CH_PD
- U1 pad 4: /WOES -> /GPIO16
Routing:
- net /DTR: track 49.3 -> 0.00 mm
- net /WOES: track 24.1 -> 0.00 mm
- net VCC: track 115.2 -> 98.3 mm, vias 6 -> 4
- net /RESET: track 0.00 -> 8.95 mm
- net /CH_PD: track 0.00 -> 8.08 mm
- net Net-(R3-Pad2): track 5.32 -> 0.00 mm
- net /GPIO9: track 4.24 -> 0.00 mm
- net /GPIO10: track 4.15 -> 0.00 mm
- net GND: track 70.2 -> 66.2 mm
- net Net-(J2-Pad1): track 9.27 -> 10.8 mm, vias 0 -> 1
- net /GPIO14: track 51.3 -> 50.0 mm
- net /GPIO0: track 15.3 -> 14.3 mm
- net /GPIO12: track 46.8 -> 45.8 mm
- net /OUT4: track 14.2 -> 14.9 mm
- net Net-(U1-Pad19): track 0.00 -> 0.53 mm
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Other:
- board size 95.6 x 64.8 mm -> 64.8 x 95.5 mm
- net class AC: via_dia 1.2 -> 1.6
- net class Default: clearance 0.508 -> 0.2; via_dia 1.2 -> 1.6
- net class Power: clearance 0.508 -> 0.2; trace_width 0.762 -> 0.508; via_dia 1.2 -> 1.6
- rule trace_clearance: 0.508 -> 0.2
- board text added: "Blinds Controller 2018-08-01 Rev 3"
- board text added: "CH_PD"
- board text added: "DOWN"
- board text added: "GPIO0"
- board text added: "POW"
- board text added: "RST"
- board text added: "UP"
- board text removed: "Blinds Controller 2018-07-08 Rev 2"
- board text removed: "CTS"
- board text removed: "DTR"
