File: relays-hw/blinds.sch (KiCad schematic (older format))
At the start: 21 parts, among them J1 AC, J10 DC, J11 DTR, J12 DC, J2 DC, J4 SWITCH, J7 DRIVE, J8 CTS, J9 SERIAL, U1 ESP-12E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

Commit message: Revision 3
Parts:
- removed J4: SWITCH, Pin_Headers:Pin_Header_Straight_1x03_Pitch2.54mm, symbol Conn_01x03
- removed R2: 1k, Resistors_SMD:R_0805_HandSoldering, symbol R
- added J3: CH_PD, Pin_Headers:Pin_Header_Straight_1x01_Pitch2.54mm, symbol Conn_01x01
- C2: value 100nF -> 100uF
- J11: value DTR -> CH_PD
- J8: value CTS -> GPIO0
- R1: value 1k -> 10k
- U2: footprint footprints:LB1909MC_W -> footprints:LB1909MC
Connections:
- net labels added: CH_PD, GPIO15, GPIO16, INT_LED, RESET
- net labels removed: CTS, DTR, GPIO10, GPIO9, LED, WOES
- wire segments 71 -> 61
Other:
- moved on the sheet: R1
Changed lines of the file:
@@
 LIBS:ESP8266
 LIBS:w_relay
-LIBS:conn
+LIBS:blinds-cache
 LIBS:Connector_Generic_MountingPin
 LIBS:Connector_Generic_Shielded
 LIBS:Connector_Generic
 LIBS:Connector
-LIBS:Converter_ACDC
-LIBS:modules
 LIBS:power
 LIBS:powerint
@@
 F 0 "U2" H 2800 2350 50  0000 L CNN
 F 1 "LB1909MC" H 2800 1650 50  0000 L CNN
-F 2 "footprints:LB1909MC_W" H 3100 1450 50  0001 C CNN
+F 2 "footprints:LB1909MC" H 3100 1450 50  0001 C CNN
 F 3 "" H 2800 2350 50  0001 C CNN
 	1    3100 2000
@@
 	1    0    0    -1
 $EndComp
-Text Label 6100 1000 0    60   ~ 0
-VCC
 $Comp
 L R R4
@@
 	-1   0    0    1
 $EndComp
-Text Label 9350 2050 0    60   ~ 0
-VCC
 Text Label 8700 2050 0    60   ~ 0
 TXD
@@
 	6600 2250 6900 2250
 Wire Wire Line
-	8700 2450 9550 2450
-Wire Wire Line
 	8700 2050 8950 2050
 Wire Wire Line
 	8700 2150 8950 2150
-Connection ~ 9250 2450
 Wire Wire Line
 	6900 2350 6650 2350
@@
 	6900 2650 6650 2650
 Wire Wire Line
-	7750 3250 7750 3500
-Wire Wire Line
-	7850 3250 7850 3500
-Wire Wire Line
 	8700 2250 8950 2250
 Wire Wire Line
 	8700 2350 8950 2350
-Text Label 7750 3500 1    60   ~ 0
-GPIO9
-Text Label 7850 3500 1    60   ~ 0
-GPIO10
 Text Label 8700 2250 0    60   ~ 0
 GPIO5
@@
 GPIO0
 Text Label 6650 2350 0    60   ~ 0
-WOES
+GPIO16
 Text Label 6650 2450 0    60   ~ 0
 GPIO14
@@
 L R R1
 U 1 1 5B2D695A
-P 6600 1900
-F 0 "R1" V 6680 1900 50  0000 C CNN
-F 1 "1k" V 6600 1900 50  0000 C CNN
-F 2 "Resistors_SMD:R_0805_HandSoldering" V 6530 1900 50  0001 C CNN
-F 3 "" H 6600 1900 50  0001 C CNN
-	1    6600 1900
-	-1   0    0    1
+P 6450 2050
+F 0 "R1" V 6530 2050 50  0000 C CNN
+F 1 "10k" V 6450 2050 50  0000 C CNN
+F 2 "Resistors_SMD:R_0805_HandSoldering" V 6380 2050 50  0001 C CNN
+F 3 "" H 6450 2050 50  0001 C CNN
+	1    6450 2050
+	0    -1   -1   0
 $EndComp
 $Comp
@@
 	6900 2050 6600 2050
 Wire Wire Line
-	6300 1000 6300 2750
+	6300 1600 6300 2750
 Connection ~ 6300 2250
-Text Label 9350 3250 0    60   ~ 0
-GND
 $Comp
 L R R5
@@
 $EndComp
 Wire Wire Line
-	9250 2150 9250 2050
-Wire Wire Line
-	9250 2050 9550 2050
+	9250 1600 9250 2150
 Wire Wire Line
 	8700 2650 9250 2650
-Wire Wire Line
-	8700 2750 8700 3250
 Wire Wire Line
 	9150 4550 8850 4550
@@
 	9150 4200 8850 4200
 Text Label 8850 4650 0    60   ~ 0
-DTR
+CH_PD
 Text Label 8850 4000 0    60   ~ 0
 RXD
@@
 VCC
 Text Label 8850 4550 0    60   ~ 0
-CTS
+GPIO0
 Text Label 8850 4300 0    60   ~ 0
 GND
-Text Label 6650 2050 0    60   ~ 0
-DTR
-Text Label 9350 2450 0    60   ~ 0
-CTS
-Wire Wire Line
-	8700 3250 9550 3250
 $Comp
 L C C1
@@
 Wire Wire Line
 	6300 3050 6300 3200
-Wire Wire Line
-	6300 3200 6100 3200
-Text Label 6100 3200 0    60   ~ 0
-GND
-Wire Wire Line
-	9250 2950 9250 3250
-Connection ~ 9250 3250
-$Comp
-L Conn_01x03 J4
-U 1 1 5B2D8A84
-P 8300 4100
-F 0 "J4" H 8300 4300 50  0000 C CNN
-F 1 "SWITCH" H 8300 3900 50  0000 C CNN
-F 2 "Pin_Headers:Pin_Header_Straight_1x03_Pitch2.54mm" H 8300 4100 50  0001 C CNN
-F 3 "" H 8300 4100 50  0001 C CNN
-	1    8300 4100
-	1    0    0    -1
-$EndComp
-Wire Wire Line
-	8100 4000 7750 4000
-Wire Wire Line
-	8100 4100 7750 4100
-Wire Wire Line
-	8100 4200 7750 4200
-Text Label 7750 4000 0    60   ~ 0
-VCC
 $Comp
 L Screw_Terminal_01x03 J7
@@
 Wire Wire Line
 	3000 5800 3000 5850
-Text Label 7750 4200 0    60   ~ 0
-GPIO10
-Text Label 7750 4100 0    60   ~ 0
-GPIO9
 Wire Wire Line
 	2300 2950 2750 2950
@@
 	8700 2550 8950 2550
 Text Label 8700 2550 0    60   ~ 0
-LED
+INT_LED
 Connection ~ 9250 2650
 $Comp
@@
 P 9350 4650
 F 0 "J11" H 9350 4750 50  0000 C CNN
-F 1 "DTR" H 9350 4550 50  0000 C CNN
+F 1 "CH_PD" H 9350 4550 50  0000 C CNN
 F 2 "Pin_Headers:Pin_Header_Straight_1x01_Pitch2.54mm" H 9350 4650 50  0001 C CNN
 F 3 "" H 9350 4650 50  0001 C CNN
@@
 P 9350 4550
 F 0 "J8" H 9350 4650 50  0000 C CNN
-F 1 "CTS" H 9350 4450 50  0000 C CNN
+F 1 "GPIO0" H 9350 4450 50  0000 C CNN
 F 2 "Pin_Headers:Pin_Header_Straight_1x01_Pitch2.54mm" H 9350 4550 50  0001 C CNN
 F 3 "" H 9350 4550 50  0001 C CNN
@@
 GPIO4
 $Comp
-L R R2
-U 1 1 5B315448
-P 6600 1500
-F 0 "R2" V 6680 1500 50  0000 C CNN
-F 1 "1k" V 6600 1500 50  0000 C CNN
-F 2 "Resistors_SMD:R_0805_HandSoldering" V 6530 1500 50  0001 C CNN
-F 3 "" H 6600 1500 50  0001 C CNN
-	1    6600 1500
-	-1   0    0    1
-$EndComp
-Wire Wire Line
-	6600 1750 6600 1650
-Wire Wire Line
-	6100 1000 6600 1000
-Wire Wire Line
-	6600 1000 6600 1350
-Connection ~ 6300 1000
-Wire Wire Line
-	6600 1700 6900 1700
-Connection ~ 6600 1700
-Text Label 6650 1700 0    60   ~ 0
-WOES
-$Comp
 L C C2
 U 1 1 5B315EA7
 P 1600 1950
 F 0 "C2" H 1625 2050 50  0000 L CNN
-F 1 "100nF" H 1625 1850 50  0000 L CNN
+F 1 "100uF" H 1625 1850 50  0000 L CNN
 F 2 "Capacitors_SMD:C_0805_HandSoldering" H 1638 1800 50  0001 C CNN
 F 3 "" H 1600 1950 50  0001 C CNN
@@
 	1    0    0    -1
 $EndComp
+Connection ~ 6300 2050
+Text Label 6650 2250 0    60   ~ 0
+CH_PD
+Text Label 8700 2650 0    60   ~ 0
+GPIO15
+Text Label 6650 2050 0    60   ~ 0
+RESET
+Wire Wire Line
+	8700 2450 9250 2450
+$Comp
+L Conn_01x01 J3
+U 1 1 5B61D4A9
+P 9350 4750
+F 0 "J3" H 9350 4850 50  0000 C CNN
+F 1 "CH_PD" H 9350 4650 50  0000 C CNN
+F 2 "Pin_Headers:Pin_Header_Straight_1x01_Pitch2.54mm" H 9350 4750 50  0001 C CNN
+F 3 "" H 9350 4750 50  0001 C CNN
+	1    9350 4750
+	1    0    0    -1
+$EndComp
+Wire Wire Line
+	9150 4750 8850 4750
+Text Label 8850 4750 0    60   ~ 0
+RESET
+$Comp
+L GND #PWR?
+U 1 1 5B678C47
+P 6300 3200
+F 0 "#PWR?" H 6300 2950 50  0001 C CNN
+F 1 "GND" H 6300 3050 50  0000 C CNN
+F 2 "" H 6300 3200 50  0001 C CNN
+F 3 "" H 6300 3200 50  0001 C CNN
+	1    6300 3200
+	1    0    0    -1
+$EndComp
+$Comp
+L VCC #PWR?
+U 1 1 5B678D1D
+P 6300 1600
+F 0 "#PWR?" H 6300 1450 50  0001 C CNN
+F 1 "VCC" H 6300 1750 50  0000 C CNN
+F 2 "" H 6300 1600 50  0001 C CNN
+F 3 "" H 6300 1600 50  0001 C CNN
+	1    6300 1600
+	1    0    0    -1
+$EndComp
+$Comp
+L VCC #PWR?
+U 1 1 5B678E86
+P 9250 1600
+F 0 "#PWR?" H 9250 1450 50  0001 C CNN
+F 1 "VCC" H 9250 1750 50  0000 C CNN
+F 2 "" H 9250 1600 50  0001 C CNN
+F 3 "" H 9250 1600 50  0001 C CNN
+	1    9250 1600
+	1    0    0    -1
+$EndComp
+$Comp
+L GND #PWR?
+U 1 1 5B678F62
+P 9250 3200
+F 0 "#PWR?" H 9250 2950 50  0001 C CNN
+F 1 "GND" H 9250 3050 50  0000 C CNN
+F 2 "" H 9250 3200 50  0001 C CNN
+F 3 "" H 9250 3200 50  0001 C CNN
+	1    9250 3200
+	1    0    0    -1
+$EndComp
+Wire Wire Line
+	9250 2950 9250 3200
+Wire Wire Line
+	8700 2750 8700 3100
+Wire Wire Line
+	8700 3100 9250 3100
+Connection ~ 9250 3100
 $EndSCHEMATC
